Commit message: wip - set the right directory for atlas package

File: robot_models/drc_atlas/drc_atlas_description/urdf/atlas_convex_hull.urdf (robot description, URDF)
Before this commit: robot atlas, 70 links, 69 joints
Links:
- link head: geometry collision mesh filename=package://drc_atlas_description/meshes/head_chull.obj; visual mesh filename=package://drc_atlas_description/meshes/head.gltf
- link hokuyo_link: geometry collision mesh filename=package://drc_atlas_description/meshes/head_camera_chull.obj; visual mesh filename=package://drc_atlas_description/meshes/head_camera.gltf
- link l_clav: geometry collision mesh filename=package://drc_atlas_description/meshes/r_clav_chull.obj; visual mesh filename=package://drc_atlas_description/meshes/r_clav.gltf
- link l_foot: geometry collision mesh filename=package://drc_atlas_description/meshes/l_foot_chull.obj; collision sphere radius=0.0
- link l_larm: geometry collision mesh filename=package://drc_atlas_description/meshes/r_larm_chull.obj; visual mesh filename=package://drc_atlas_description/meshes/r_larm.gltf
- link l_lfarm: geometry collision mesh filename=package://drc_atlas_description/meshes/r_hand_chull.obj; visual mesh filename=package://drc_atlas_description/meshes/r_hand.gltf
- link l_lglut: geometry collision mesh filename=package://drc_atlas_description/meshes/l_lglut_chull.obj; visual mesh filename=package://drc_atlas_description/meshes/l_lglut.gltf
- link l_lleg: geometry collision mesh filename=package://drc_atlas_description/meshes/l_lleg_chull.obj; visual mesh filename=package://drc_atlas_description/meshes/l_lleg.gltf
- link l_scap: geometry collision mesh filename=package://drc_atlas_description/meshes/r_scap_chull.obj; visual mesh filename=package://drc_atlas_description/meshes/r_scap.gltf
- link l_talus: geometry visual mesh filename=package://drc_atlas_description/meshes/l_talus.gltf
- link l_uarm: geometry collision mesh filename=package://drc_atlas_description/meshes/r_uarm_chull.obj; visual mesh filename=package://drc_atlas_description/meshes/r_uarm.gltf
- link l_ufarm: geometry collision mesh filename=package://drc_atlas_description/meshes/r_farm_chull.obj; visual mesh filename=package://drc_atlas_description/meshes/r_farm.gltf
- link l_uglut: geometry collision mesh filename=package://drc_atlas_description/meshes/l_uglut_chull.obj; visual mesh filename=package://drc_atlas_description/meshes/l_uglut.gltf
- link l_uleg: geometry collision mesh filename=package://drc_atlas_description/meshes/l_uleg_chull.obj; visual mesh filename=package://drc_atlas_description/meshes/l_uleg.gltf
- link left_palm: geometry collision mesh filename=package://drc_atlas_description/meshes/GRIPPER_OPEN_chull.o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 scale=1 1 1; visual mesh filename=package://drc_atlas_description/meshes/GRIPPER_OPEN_chull.g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 scale=1 1 1
- link ltorso: geometry visual mesh filename=package://drc_atlas_description/meshes/ltorso.gltf
- link mtorso: geometry visual mesh filename=package://drc_atlas_description/meshes/mtorso.gltf
- link pelvis: geometry collision mesh filename=package://drc_atlas_description/meshes/pelvis_chull.obj; visual mesh filename=package://drc_atlas_description/meshes/pelvis.gltf
- link r_clav: geometry collision mesh filename=package://drc_atlas_description/meshes/r_clav_chull.obj; visual mesh filename=package://drc_atlas_description/meshes/r_clav.gltf
- link r_foot: geometry collision mesh filename=package://drc_atlas_description/meshes/r_foot_chull.obj; collision sphere radius=0.0
- link r_larm: geometry collision mesh filename=package://drc_atlas_description/meshes/r_larm_chull.obj; visual mesh filename=package://drc_atlas_description/meshes/r_larm.gltf
- link r_lfarm: geometry collision mesh filename=package://drc_atlas_description/meshes/r_hand_chull.obj; visual mesh filename=package://drc_atlas_description/meshes/r_hand.gltf
- link r_lglut: geometry collision mesh filename=package://drc_atlas_description/meshes/r_lglut_chull.obj; visual mesh filename=package://drc_atlas_description/meshes/r_lglut.gltf
- link r_lleg: geometry collision mesh filename=package://drc_atlas_description/meshes/r_lleg_chull.obj; visual mesh filename=package://drc_atlas_description/meshes/r_lleg.gltf
- link r_scap: geometry collision mesh filename=package://drc_atlas_description/meshes/r_scap_chull.obj; visual mesh filename=package://drc_atlas_description/meshes/r_scap.gltf
- link r_talus: geometry visual mesh filename=package://drc_atlas_description/meshes/r_talus.gltf
- link r_uarm: geometry collision mesh filename=package://drc_atlas_description/meshes/r_uarm_chull.obj; visual mesh filename=package://drc_atlas_description/meshes/r_uarm.gltf
- link r_ufarm: geometry collision mesh filename=package://drc_atlas_description/meshes/r_farm_chull.obj; visual mesh filename=package://drc_atlas_description/meshes/r_farm.gltf
- link r_uglut: geometry collision mesh filename=package://drc_atlas_description/meshes/r_uglut_chull.obj; visual mesh filename=package://drc_atlas_description/meshes/r_uglut.gltf
- link r_uleg: geometry collision mesh filename=package://drc_atlas_description/meshes/r_uleg_chull.obj; visual mesh filename=package://drc_atlas_description/meshes/r_uleg.gltf
- link right_palm: geometry collision mesh filename=package://drc_atlas_description/meshes/GRIPPER_OPEN_chull.o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 scale=1 1 1; visual mesh filename=package://drc_atlas_description/meshes/GRIPPER_OPEN_chull.g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 scale=1 1 1
- link utorso: geometry collision mesh filename=package://drc_atlas_description/meshes/utorso_chull.obj; visual mesh filename=package://drc_atlas_description/meshes/utorso.gltf

File: robot_models/drc_atlas/drc_atlas_description/urdf/atlas_minimal_contact.urdf (robot description, URDF)
Before this commit: robot atlas, 60 links, 59 joints
Links:
- link head: geometry visual mesh filename=package://drc_atlas_description/meshes/head.gltf
- link hokuyo_link: geometry visual mesh filename=package://drc_atlas_description/meshes/head_camera.gltf
- link l_clav: geometry visual mesh filename=package://drc_atlas_description/meshes/r_clav.gltf
- link l_foot: geometry collision sphere radius=0.0; collision sphere radius=0.0
- link l_larm: geometry visual mesh filename=package://drc_atlas_description/meshes/r_larm.gltf
- link l_lfarm: geometry visual mesh filename=package://drc_atlas_description/meshes/r_hand.gltf
- link l_lglut: geometry visual mesh filename=package://drc_atlas_description/meshes/l_lglut.gltf
- link l_lleg: geometry visual mesh filename=package://drc_atlas_description/meshes/l_lleg.gltf
- link l_scap: geometry visual mesh filename=package://drc_atlas_description/meshes/r_scap.gltf
- link l_talus: geometry visual mesh filename=package://drc_atlas_description/meshes/l_talus.gltf
- link l_uarm: geometry visual mesh filename=package://drc_atlas_description/meshes/r_uarm.gltf
- link l_ufarm: geometry visual mesh filename=package://drc_atlas_description/meshes/r_farm.gltf
- link l_uglut: geometry visual mesh filename=package://drc_atlas_description/meshes/l_uglut.gltf
- link l_uleg: geometry visual mesh filename=package://drc_atlas_description/meshes/l_uleg.gltf
- link ltorso: geometry visual mesh filename=package://drc_atlas_description/meshes/ltorso.gltf
- link mtorso: geometry visual mesh filename=package://drc_atlas_description/meshes/mtorso.gltf
- link pelvis: geometry visual mesh filename=package://drc_atlas_description/meshes/pelvis.gltf
- link r_clav: geometry visual mesh filename=package://drc_atlas_description/meshes/r_clav.gltf
- link r_foot: geometry collision sphere radius=0.0; collision sphere radius=0.0
- link r_larm: geometry visual mesh filename=package://drc_atlas_description/meshes/r_larm.gltf
- link r_lfarm: geometry visual mesh filename=package://drc_atlas_description/meshes/r_hand.gltf
- link r_lglut: geometry visual mesh filename=package://drc_atlas_description/meshes/r_lglut.gltf
- link r_lleg: geometry visual mesh filename=package://drc_atlas_description/meshes/r_lleg.gltf
- link r_scap: geometry visual mesh filename=package://drc_atlas_description/meshes/r_scap.gltf
- link r_talus: geometry visual mesh filename=package://drc_atlas_description/meshes/r_talus.gltf
- link r_uarm: geometry visual mesh filename=package://drc_atlas_description/meshes/r_uarm.gltf
- link r_ufarm: geometry visual mesh filename=package://drc_atlas_description/meshes/r_farm.gltf
- link r_uglut: geometry visual mesh filename=package://drc_atlas_description/meshes/r_uglut.gltf
- link r_uleg: geometry visual mesh filename=package://drc_atlas_description/meshes/r_uleg.gltf
- link utorso: geometry visual mesh filename=package://drc_atlas_description/meshes/utorso.gltf
