Commit message: Switch to using absl log instead of std::cerr, std::cout

File: robot_models/engineai_sa01/engineai_sa01_description/urdf/zq_sa01.urdf (robot description, URDF)
Before this commit: robot zqsa01, 13 links, 12 joints
Links:
- link base_link: geometry collision box size=0.2 0.2 0.3; visual mesh filename=package://engineai_sa01_description/meshes/Base_link.STL
- link leg_l1_link: geometry visual mesh filename=package://engineai_sa01_description/meshes/LeftLeg_Link_01.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
- link leg_l2_link: geometry visual mesh filename=package://engineai_sa01_description/meshes/LeftLeg_Link_02.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
- link leg_l3_link: geometry collision box size=0.08 0.08 0.25; visual mesh filename=package://engineai_sa01_description/meshes/LeftLeg_Link_03.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
- link leg_l4_link: geometry collision box size=0.05 0.05 0.28; visual mesh filename=package://engineai_sa01_description/meshes/LeftLeg_Link_04.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
- link leg_l5_link: geometry visual mesh filename=package://engineai_sa01_description/meshes/LeftLeg_Link_05.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
- link leg_l6_link: geometry collision mesh filename=package://engineai_sa01_description/meshes/LeftLeg_Link_06.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; visual mesh filename=package://engineai_sa01_description/meshes/LeftLeg_Link_06.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
- link leg_r1_link: geometry visual mesh filename=package://engineai_sa01_description/meshes/RightLeg_Link_01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
- link leg_r2_link: geometry visual mesh filename=package://engineai_sa01_description/meshes/RightLeg_Link_02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
- link leg_r3_link: geometry collision box size=0.08 0.08 0.25; visual mesh filename=package://engineai_sa01_description/meshes/RightLeg_Link_03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
- link leg_r4_link: geometry collision box size=0.05 0.05 0.28; visual mesh filename=package://engineai_sa01_description/meshes/RightLeg_Link_04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
- link leg_r5_link: geometry visual mesh filename=package://engineai_sa01_description/meshes/RightLeg_Link_05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
- link leg_r6_link: geometry collision mesh filename=package://engineai_sa01_description/meshes/RightLeg_Link_06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; visual mesh filename=package://engineai_sa01_description/meshes/RightLeg_Link_06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

Commit message: adds collision bodies

File: robot_models/engineai_sa01/engineai_sa01_description/urdf/zq_sa01.urdf (robot description, URDF)
Before this commit: robot zqsa01, 13 links, 12 joints
Links:
- link base_link: geometry collision box size=0.228 0.302 0.483; visual mesh filename=package://engineai_sa01_description/meshes/Base_link.STL
- link leg_l1_link: geometry collision box size=0.132 0.115 0.0608; visual mesh filename=package://engineai_sa01_description/meshes/LeftLeg_Link_01.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
- link leg_l2_link: geometry collision box size=0.125 0.059 0.1604; visual mesh filename=package://engineai_sa01_description/meshes/LeftLeg_Link_02.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
- link leg_l3_link: geometry collision cylinder length=0.3 radius=0.045; visual mesh filename=package://engineai_sa01_description/meshes/LeftLeg_Link_03.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
- link leg_l4_link: geometry collision cylinder length=0.33 radius=0.035; visual mesh filename=package://engineai_sa01_description/meshes/LeftLeg_Link_04.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
- link leg_l5_link: geometry collision sphere radius=0.0175; visual mesh filename=package://engineai_sa01_description/meshes/LeftLeg_Link_05.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
- link leg_l6_link: geometry collision sphere radius=0.01; collision sphere radius=0.01
- link leg_r1_link: geometry collision box size=0.132 0.115 0.0608; visual mesh filename=package://engineai_sa01_description/meshes/RightLeg_Link_01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
- link leg_r2_link: geometry collision box size=0.125 0.059 0.1604; visual mesh filename=package://engineai_sa01_description/meshes/RightLeg_Link_02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
- link leg_r3_link: geometry collision cylinder length=0.3 radius=0.045; visual mesh filename=package://engineai_sa01_description/meshes/RightLeg_Link_03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
- link leg_r4_link: geometry collision cylinder length=0.33 radius=0.035; visual mesh filename=package://engineai_sa01_description/meshes/RightLeg_Link_04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
- link leg_r5_link: geometry collision sphere radius=0.0175; visual mesh filename=package://engineai_sa01_description/meshes/RightLeg_Link_05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
- link leg_r6_link: geometry collision sphere radius=0.01; collision sphere radius=0.01
